Commit message: Revert to indigo.

File: turtlebot2i_description/robots/kobuki_interbotix_astra.urdf.xacro (robot description, xacro)
@@ -7,11 +7,7 @@
 -->
 <robot name="turtlebot" xmlns:xacro="http://ros.org/wiki/xacro">
-  <xacro:include filename="$(find turtlebot2i_description)/urdf/turtlebot_library.urdf.xacro" />
+  <xacro:include filename="$(find turtlebot_description)/urdf/turtlebot_library.urdf.xacro" />
   <kobuki/>
-  <stack_interbotix parent="base_link"/>
-  <sensor_astra parent="base_link"/>
-  <sensor_sr300 parent="base_link"/>
-  <phantomx_pincher_arm parent="base_link" color="Red" gripper_color="Red">
-    <origin xyz="0.145 0.0 0.112"/>
-  </phantomx_pincher_arm>
+  <stack_hexagons                 parent="base_link"/>
+  <sensor_asus_xtion_pro          parent="base_link"/>
 </robot>

Commit message: Adjust URDF files for Gazebo.

File: turtlebot2i_description/robots/kobuki_interbotix_astra.urdf.xacro (robot description, xacro)
@@ -7,7 +7,11 @@
 -->
 <robot name="turtlebot" xmlns:xacro="http://ros.org/wiki/xacro">
-  <xacro:include filename="$(find turtlebot_description)/urdf/turtlebot_library.urdf.xacro" />
+  <xacro:include filename="$(find turtlebot2i_description)/urdf/turtlebot_library.urdf.xacro" />
   <kobuki/>
-  <stack_hexagons                 parent="base_link"/>
-  <sensor_asus_xtion_pro          parent="base_link"/>
+  <stack_interbotix parent="base_link"/>
+  <sensor_astra parent="base_link"/>
+  <sensor_sr300 parent="base_link"/>
+  <phantomx_pincher_arm parent="base_link" color="Red" gripper_color="Red">
+    <origin xyz="0.145 0.0 0.112"/>
+  </phantomx_pincher_arm>
 </robot>

File: turtlebot2i_description/robots/kobuki_interbotix_zr300.urdf.xacro (robot description, xacro)
@@ -12,4 +12,5 @@
   <sensor_zr300 parent="base_link"/>
   <sensor_sr300 parent="base_link"/>
+<!---->
   <phantomx_pincher_arm parent="base_link" color="Red" gripper_color="Red">
     <origin xyz="0.145 0.0 0.112"/>

File: turtlebot2i_description/urdf/sensors/sr300.urdf.xacro (robot description, xacro)
@@ -38,5 +38,5 @@
         <origin xyz="0.0 0.0 0.0" rpy="0 0 0"/>
         <geometry>
-          <mesh filename="package://turtlebot2i_description/meshes/sensors/sr300.stl" scale="2.0 2.0 2.0" />
+          <mesh filename="package://turtlebot2i_description/meshes/sensors/sr300.stl" scale="1.5 1.5 1.5" />
         </geometry>
       </collision>

File: turtlebot2i_description/urdf/stacks/interbotix.urdf.xacro (robot description, xacro)
@@ -198,5 +198,6 @@
         <origin xyz="0 0 0" rpy="0 0 0"/>
         <geometry>
-          <cylinder length="0.006" radius="0.170"/>
+          <mesh filename="package://turtlebot2i_description/meshes/stacks/interbotix/TurtleBot2i_BottomPlate.stl"/>
+          <!--<cylinder length="0.006" radius="0.170"/-->
         </geometry>
       </collision>
@@ -237,4 +238,5 @@
         <geometry>
           <mesh filename="package://turtlebot2i_description/meshes/stacks/interbotix/TurtleBot2i_MiddlePlate.stl"/>
+          <!--<cylinder length="0.006" radius="0.170"/>-->
         </geometry>
       </collision>
@@ -273,4 +275,5 @@
         <geometry>
           <mesh filename="package://turtlebot2i_description/meshes/stacks/interbotix/TurtleBot2i_CameraPlate.stl"/>
+          <!--<cylinder length="0.006" radius="0.170"/>-->
         </geometry>
       </collision>
@@ -309,4 +312,5 @@
         <geometry>
           <mesh filename="package://turtlebot2i_description/meshes/stacks/interbotix/TurtleBot2i_UtilityPlate.stl"/>
+          <!--<cylinder length="0.006" radius="0.170"/>-->
         </geometry>
       </collision>
@@ -342,7 +346,8 @@
       </visual>
       <collision>
-        <origin xyz="0 0 0" rpy="0 0 0"/>
-        <geometry>
           <mesh filename="package://turtlebot2i_description/meshes/stacks/interbotix/TurtleBot2i_TopPlate.stl"/>
+        <!--<origin xyz="0 0 0" rpy="0 0 0"/>-->
+        <geometry>
+          <cylinder length="0.006" radius="0.170"/>
         </geometry>
       </collision>

File: turtlebot2i_description/urdf/turtlebot_gazebo.urdf.xacro (robot description, xacro)
@@ -1,8 +1,9 @@
 <?xml version="1.0"?>
 <robot name="turtlebot_gazebo" xmlns:xacro="http://ros.org/wiki/xacro">
+  <!-- ros_control plugin -->
   <gazebo>
-    <plugin filename="libgazebo_ros_control.so" name="gazebo_ros_control">
-        <robotNamespace>/turtlebot</robotNamespace>
-        <robotSimType>gazebo_ros_control/DefaultRobotHWSim</robotSimType>
+    <plugin name="gazebo_ros_control" filename="libgazebo_ros_control.so">
+      <robotNamespace>/turtlebot</robotNamespace>
+      <robotSimType>gazebo_ros_control/DefaultRobotHWSim</robotSimType>
     </plugin>
   </gazebo>

File: turtlebot2i_description/urdf/turtlebot_library.urdf.xacro (robot description, xacro)
@@ -17,3 +17,5 @@
   <!-- Arms -->
   <xacro:include filename="$(find turtlebot2i_description)/urdf/arms/phantomx_pincher_arm.urdf.xacro"/>
+  <!-- Gazebo controller -->
+  <xacro:include filename="$(find turtlebot2i_description)/urdf/gazebo_controller.urdf.xacro"/>
 </robot>
